File: circuit/circuit.sch (EAGLE design)
At the start: 8 parts

Commit message: update
Parts:
- added C2, C3: 100u, my:CE-16V-06.3-5.08
- added C4, C5: 0.1u, my:C-50V-0302-2.54
- added C6: 220u, my:CE-16V-04-2.54
- added D5: (no value), diode:SCHOTTKY-DIODEDO35-7
- added D6, D7, D8, D9: 1N4148DO35-7, diode:1N4148DO35-7
- added G1, G2: NiMH, battery:CRAA
- added IC1: ESP-WROOM-02, my:ESP-WROOM-02
- added IC2: 4066N, 40xx:4066N
- added L1: 47u, rcl:L-US6000-XXX-RC
- added R10: 10 1%, my:R-1/4W-07.62
- added R11, R3, R4, R5, R6, R7: 10k, my:R-1/4W-07.62
- added R8: 200k, my:R-1/4W-07.62
- added R9: 100k, my:R-1/4W-07.62
- added S1: RESET, SparkFun-Electromechanical:TAC_SWITCHPTH
- added S2: PROGRAM, SparkFun-Electromechanical:TAC_SWITCHPTH
- added U$1: HT77XXAT, my:HT77XXAT
- added U$2: MCP3425, my:MCP3425
- added U2: (no value), SparkFun-Connectors:AUDIO-JACK2.5MM
- C1: value 10u -> 220u
Connections:
- new net 3.3V: C3.+, C4.1, C5.1, D5.C, IC1.3V3, IC2P.VDD, R3.2, R4.1, R6.1, R7.2, U$1.VOUT, U$2.VDD
- new net BAT_ADC: IC1.TOUT, R8.2, R9.1
- new net CTRL_CH1: IC1.IO12, IC2A.C
- new net CTRL_CH2: IC1.IO13, IC2B.C
- new net N$10: G1.-, G2.+
- new net N$11: D5.A, L1.2, U$1.LX
- new net N$12: D6.A, D7.C, U2.LEFT
- new net N$13: C2.+, G1.+, L1.1, R8.1
- new net N$14: IC2A.A, IC2B.A, U$2.VIN+
- new net N$15: D8.A, D9.C, U2.SLEEVE
- new net N$16: D6.C, D8.C, R10.2, R11.2
- new net N$17: C6.+, IC2B.B, R11.1
- new net N$2: IC1.EN, R3.1
- new net N$6: IC1.IO15, R5.1
- new net N$7: IC1.IO2, R7.1
- new net N$8: IC1.IO0, R4.2, S2.1, S2.2
- new net N$9: IC1.RST, R6.2, S1.1, S1.2
- new net RXD: IC1.RXD
- new net SCL: IC1.IO5, U$2.SCL
- new net SDA: IC1.IO4, U$2.SDA
- new net TXD: IC1.TXD
- net GND: now also C2.-, C3.-, C4.2, C5.2, C6.-, D7.A, D9.A, G2.-, IC1.GND1, IC1.GND2, IC1.GND3, IC2P.VSS, R10.1, R5.2, R9.2, S1.3, S1.4, S2.3, S2.4, U$1.GND, U$2.VIN-, U$2.VSS
- net N$1: now also IC2A.B
Other:
- note added: "2.4V TO 3.3V STEP-UP"
- note added: "CURRENT TRANSFORMER"
- moved on the sheet: C1, D1, D2, D3, D4, R1, R2, U1
